File: OMC_WIFI_PCB/V1.6/OMC_WIFI_PCB.sch (KiCad schematic (older format))
At the start: 26 parts, among them J1 Conn_01x02_Male, J10 Conn_01x01_Male, J2 Conn_01x02_Female, J3 Conn_01x02_Male, J4 Switch, J5 Pins_FT232R, J6 Level shifter, J7 Conn_01x01_Female, J8 Regulador, J9 Conn_01x01_Female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

Commit message: Creación de versión 1.6 PCB
Parts:
- K1: symbol OMC_WIFI_PCB-rescue:SLA-12VDC-SL-C-SLA-12VDC-SL-C -> SLA-12VDC-SL-C:SLA-12VDC-SL-C
- U2: symbol OMC_WIFI_PCB-rescue:PZEM-004T-100A-omc-schematics -> omc-schematics:PZEM-004T-100A
Connections:
- net EN is gone; now on an unnamed net: U1.3 (EN)
- net +3V: now also U1.2 (VDD)
- net at C1.1, R4.2: no longer U1.2 (VDD)
- net D22_LED_G renamed D23_LED_G
- net D23_LED_R renamed D22_LED_R
- net D32_RELAY_3V: no longer names the net of J6.9 (Pin_9)
- net D32_RELAY_3V: no longer U1.33 (IO21)
- net D32_RELAY_5V: no longer names the net of J6.10 (Pin_10)
- net D32_RELAY_5V: no longer R3.1
- new net D21_RELAY: R3.1, U1.33 (IO21)
- no-connect marks 29 -> 31
Other:
- note added: "ESP-WROOM-32\n"
- note added: "Touch"
- note removed: "Microcontrolador"
- note removed: "Módulo ESP-WROOM32\n"
- moved on the sheet: C1, D1, D2, J3, J5, R1, R2, R4, U1
